File: hedge65-pcb/_autosave-hedge65-pcb.kicad_pcb (KiCad board)
At the start: 2 copper layers, 164 parts, among them J1 USB_C_Receptacle_USB2.0, SW1 SW_PUSH, U1 ATmega32U4-AU, Y1 16MHz

Commit message: redo
Parts:
- C1: renamed from C2; moved to F.Cu
- C2: renamed from C3; moved to F.Cu
- C6: renamed from C5; moved to B.Cu
- F1, J1: moved to B.Cu
- moved J1 123.9 mm to (27.9, 116.8)
- moved R5 67.4 mm to (25.4, 138.4)
- moved F1 55.4 mm to (21.6, 146.1), turned to 270 degrees
- moved R3 53.9 mm to (41.9, 149.9)
- moved SW1 53.6 mm to (58.4, 162.6)
- moved C3 43.2 mm to (47.0, 139.7), turned to 90 degrees
- moved C6 33.3 mm to (63.5, 151.1), turned to 180 degrees
- moved R4 32.6 mm to (67.3, 144.8)
- moved R2 30.2 mm to (44.5, 144.8)
- moved R6 28.1 mm to (110.5, 154.9)
- moved C4 28.0 mm to (14.0, 132.1), turned to 90 degrees
- moved C7 25.3 mm to (67.3, 135.9), turned to 90 degrees
- moved C5 22.7 mm to (20.3, 132.1), turned to 90 degrees
- moved C1 5.68 mm to (62.2, 125.7)
- moved C2 2.54 mm to (52.1, 125.7), turned to 90 degrees
- renumbered C6 to C3, C1 to C4, C4 to C5, R3 to R1, R1 to R3
Connections:
- U1 pad 10: Net-(U1-Pad10) -> row2
- U1 pad 11: Net-(U1-Pad11) -> row3
- U1 pad 12: Net-(U1-Pad12) -> col2
- U1 pad 18: Net-(U1-Pad18) -> col5
- U1 pad 19: Net-(U1-Pad19) -> col6
- U1 pad 20: Net-(U1-Pad20) -> col7
- U1 pad 21: Net-(U1-Pad21) -> col8
- U1 pad 22: Net-(U1-Pad22) -> col10
- U1 pad 25: Net-(U1-Pad25) -> col9
- U1 pad 26: Net-(U1-Pad26) -> col11
- U1 pad 27: Net-(U1-Pad27) -> col12
- U1 pad 28: Net-(U1-Pad28) -> row4
- U1 pad 29: Net-(U1-Pad29) -> col0
- U1 pad 30: Net-(U1-Pad30) -> col1
- U1 pad 31: Net-(U1-Pad31) -> col3
- U1 pad 32: Net-(U1-Pad32) -> col4
- U1 pad 39: Net-(U1-Pad39) -> col15
- U1 pad 40: Net-(U1-Pad40) -> col14
- U1 pad 41: Net-(U1-Pad41) -> col13
- U1 pad 8: Net-(U1-Pad8) -> row0
- U1 pad 9: Net-(U1-Pad9) -> row1
