File: hedge65-pcb/hedge65-pcb.kicad_pcb (KiCad board)
At the start: 2 copper layers, 164 parts, among them J1 USB_C_Receptacle_USB2.0, SW1 SW_PUSH, U1 ATmega32U4-AU, Y1 16MHz

Commit message: attached diodes
Parts:
- moved D69 317.8 mm to (315.0, 25.4), turned to 90 degrees
- moved D70 315.4 mm to (315.0, 44.5), turned to 90 degrees
- moved D60 294.0 mm to (276.9, 25.4), turned to 90 degrees
- moved D64 275.5 mm to (295.9, 25.4), turned to 90 degrees
- moved D65 271.6 mm to (295.9, 44.5), turned to 90 degrees
- moved D1 270.6 mm to (29.2, 25.4), turned to 90 degrees
- moved D68 268.8 mm to (295.9, 101.6), turned to 90 degrees
- moved D67 268.3 mm to (295.9, 82.5), turned to 90 degrees
- moved D2 255.8 mm to (29.2, 44.5), turned to 90 degrees
- moved D71 254.9 mm to (315.0, 63.5), turned to 90 degrees
- moved D55 252.7 mm to (257.8, 25.4), turned to 90 degrees
- moved D3 248.5 mm to (29.2, 63.5), turned to 90 degrees
- moved D61 234.5 mm to (276.9, 44.5), turned to 90 degrees
- moved D62 230.7 mm to (276.9, 63.5), turned to 90 degrees
- moved D8 228.8 mm to (48.3, 63.5), turned to 90 degrees
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
Commit message: redo
Parts:
- C2, C3, U1, Y1: moved to B.Cu
- moved D50 261.0 mm to (238.8, 25.4), turned to 90 degrees
- moved D72 238.3 mm to (315.0, 82.5), turned to 90 degrees
- moved D38 220.6 mm to (181.6, 44.5), turned to 90 degrees
- moved D28 220.3 mm to (143.5, 25.4), turned to 90 degrees
- moved D37 219.9 mm to (181.6, 25.4), turned to 90 degrees
- moved D42 217.8 mm to (200.7, 25.4), turned to 90 degrees
- moved D6 217.2 mm to (48.3, 25.4), turned to 90 degrees
- moved D19 214.2 mm to (105.4, 25.4), turned to 90 degrees
- moved D47 205.1 mm to (219.7, 44.5), turned to 90 degrees
- moved D20 201.9 mm to (105.4, 44.5), turned to 90 degrees
- moved D39 200.8 mm to (181.6, 63.5), turned to 90 degrees
- moved D35 199.3 mm to (162.6, 63.5), turned to 90 degrees
- moved D29 197.5 mm to (143.5, 44.5), turned to 90 degrees
- moved D34 197.2 mm to (162.6, 44.5), turned to 90 degrees
- moved D43 192.3 mm to (200.7, 44.5), turned to 90 degrees
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
Commit message: doides shifted to deadspace
Parts:
- removed D32: D_Small, Diode_SMD:D_SOD-123
- removed F1: 500mA, Fuse:Fuse_1206_3216Metric
- removed R5, R6: 5.1k, Resistor_SMD:R_0805_2012Metric
- removed Y1: 16MHz, Crystal:Crystal_SMD_3225-4Pin_3.2x2.5mm
- added X1: XTAL_GND, Crystal:Crystal_SMD_3225-4Pin_3.2x2.5mm, F.Cu at (53.7, 154.4)
- C1: value 0.1uF -> 22p
- C2: value 22pF -> 22p; moved to F.Cu
- C3: value 22pF -> 0.1u; moved to F.Cu
- C4, C5: value 0.1uF -> 0.1u
- C6: value 1uF -> 0.1u
- C7: value 10uF -> 4.7u
- D1, D10, D11, D12, D13, D14, D15, D16, D17, D18, D19, D2, D20, D21, D22, D23, D24, D25, D26, D27, D28, D29, D3, D30, D31, D33, D34, D35, D36, D37, D38, D39, D4, D40, D41, D42, D43, D44, D45, D46, D47, D48, D49, D5, D50, D51, D52, D53, D54, D55, D56, D57, D58, D59, D6, D60, D61, D62, D63, D64, D65, D66, D67, D68, D69, D7, D70, D71, D72, D73, D8, D9: footprint Diode_SMD:D_SOD-123 -> cftkb:D_DO-35_SOD27_P5.08mm_Horizontal
- J1: value USB_C_Receptacle_USB2.0 -> USB_C_Receptacle; footprint Type-C:HRO-TYPE-C-31-M-12-HandSoldering -> Connector_USB:USB_C_Receptacle_Amphenol_12401548E4-2A_CircularHoles
- R1, R2: value 22 -> R_Small
- R3, R4: value 10k -> R_Small
- U1: value ATmega32U4-AU -> ATMEGA32U4; footprint Package_QFP:TQFP-44_10x10mm_P0.8mm -> ATmega32U4:ATmega32U4; moved to F.Cu
- moved U1 140.2 mm to (-80.0, 168.9)
- moved J1 104.5 mm to (47.0, 179.1)
- moved D63 88.9 mm to (274.3, 12.7)
- moved D41 88.9 mm to (180.3, 12.7)
- moved D5 88.9 mm to (27.9, 12.7)
- moved D73 88.9 mm to (316.2, 12.7)
- moved D14 88.9 mm to (67.3, 12.7)
- moved D27 88.9 mm to (124.5, 12.7)
- moved D54 88.9 mm to (238.8, 12.7)
- moved D59 88.9 mm to (257.8, 12.7)
- moved D68 88.9 mm to (295.9, 12.7)
- moved D4 70.0 mm to (24.1, 12.7)
- moved D40 70.0 mm to (176.5, 12.7)
- moved D13 70.0 mm to (63.5, 12.7)
- moved D22 70.0 mm to (101.6, 12.7)
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Connections:
- C1 pad 1: +5V -> Net-(C1-Pad1)
- C2 pad 1: +5V -> Net-(C2-Pad1)
- C2 pad 2: Net-(C2-Pad2) -> +5V
- C3 pad 1: +5V -> VCC
- C4 pad 1: +5V -> VCC
- C4 pad 2: +5V -> Net-(C3-Pad2)
- C5 pad 1: +5V -> VCC
- C5 pad 2: +5V -> Net-(C3-Pad2)
- C6 pad 1: Net-(C6-Pad1) -> VCC
- C6 pad 2: +5V -> Net-(C3-Pad2)
- C7 pad 1: +5V -> VCC
- C7 pad 2: +5V -> Net-(C3-Pad2)
- MX32 pad 1: col6 -> col8
- MX32 pad 2: Net-(D32-Pad2) -> Net-(D41-Pad2)
- R1 pad 1: D- -> +5V
- R1 pad 2: Net-(R1-Pad2) -> Net-(J1-PadA5)
- R2 pad 1: D+ -> +5V
- R2 pad 2: Net-(R2-Pad2) -> Net-(J1-PadB5)
- R3 pad 1: +5V -> Net-(R3-Pad1)
- R3 pad 2: Net-(R3-Pad2) -> VCC
- R4 pad 1: Net-(R4-Pad1) -> +5V
- R4 pad 2: +5V -> Net-(R4-Pad2)
- SW1 pad 2: Net-(R3-Pad2) -> Net-(R3-Pad1)
- U1 pad 10: Net-(U1-Pad10) -> col12
- U1 pad 11: Net-(U1-Pad11) -> col13
- U1 pad 12: Net-(U1-Pad12) -> col14
- U1 pad 13: Net-(R3-Pad2) -> Net-(R3-Pad1)
- U1 pad 14: +5V -> VCC
- U1 pad 16: Net-(C3-Pad2) -> Net-(C1-Pad1)
- U1 pad 17: Net-(C2-Pad2) -> Net-(C2-Pad1)
- U1 pad 18: Net-(U1-Pad18) -> col15
- U1 pad 2: +5V -> VCC
- U1 pad 24: +5V -> VCC
- U1 pad 25: Net-(U1-Pad25) -> col9
- U1 pad 26: Net-(U1-Pad26) -> col8
- U1 pad 27: Net-(U1-Pad27) -> col7
- U1 pad 28: Net-(U1-Pad28) -> col6
- U1 pad 29: Net-(U1-Pad29) -> col5
- U1 pad 3: Net-(R1-Pad2) -> Net-(J1-PadA7)
- U1 pad 30: Net-(U1-Pad30) -> col4
- U1 pad 31: Net-(U1-Pad31) -> col3
- U1 pad 32: Net-(U1-Pad32) -> col2
- U1 pad 33: Net-(R4-Pad1) -> Net-(R4-Pad2)
- U1 pad 34: +5V -> VCC
- U1 pad 36: Net-(U1-Pad36) -> col1
- U1 pad 37: Net-(U1-Pad37) -> row4
- U1 pad 38: Net-(U1-Pad38) -> row3
- U1 pad 39: Net-(U1-Pad39) -> row2
- U1 pad 4: Net-(R2-Pad2) -> Net-(J1-PadA6)
- U1 pad 40: Net-(U1-Pad40) -> row1
- U1 pad 41: Net-(U1-Pad41) -> row0
- U1 pad 44: +5V -> VCC
- U1 pad 6: Net-(C6-Pad1) -> Net-(U1-Pad6)
- U1 pad 7: +5V -> Net-(U1-Pad7)
- U1 pad 8: Net-(U1-Pad8) -> col10
- U1 pad 9: Net-(U1-Pad9) -> col11

Commit message: doides all flipped to 225
Parts:
- moved D53 35.1 mm to (200.7, 5.08), turned to 225 degrees
- moved D57 35.1 mm to (215.9, 5.08), turned to 225 degrees
- moved D65 34.9 mm to (250.2, 6.35), turned to 225 degrees
- moved D61 34.9 mm to (232.4, 6.35), turned to 225 degrees
- moved D69 33.6 mm to (268.0, 6.35), turned to 225 degrees
- moved D52 32.6 mm to (200.7, 1.27), turned to 225 degrees
- moved D56 32.6 mm to (215.9, 1.27), turned to 225 degrees
- moved D64 32.1 mm to (250.2, 2.54), turned to 225 degrees
- moved D60 32.1 mm to (232.4, 2.54), turned to 225 degrees
- moved D51 30.7 mm to (200.7, -2.54), turned to 225 degrees
- moved D55 30.7 mm to (215.9, -2.54), turned to 225 degrees
- moved D49 30.2 mm to (186.7, 5.08), turned to 225 degrees
- moved D73 29.9 mm to (287.0, 6.35), turned to 225 degrees
- moved D50 29.8 mm to (200.7, -6.35), turned to 225 degrees
- moved D54 29.8 mm to (215.9, -6.35), turned to 225 degrees
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
Commit message: diodes like cftkb
Parts:
- D1, D10, D11, D12, D13, D14, D15, D16, D17, D18, D19, D2, D20, D21, D22, D23, D24, D25, D26, D27, D28, D29, D3, D30, D31, D33, D34, D35, D36, D37, D38, D39, D4, D40, D41, D42, D43, D44, D45, D46, D47, D48, D49, D5, D50, D51, D52, D53, D54, D55, D56, D57, D58, D59, D6, D60, D61, D62, D63, D64, D65, D66, D67, D68, D69, D7, D70, D71, D72, D73, D8, D9: moved to B.Cu
- moved D13 26.7 mm to (39.4, -6.35), turned to 270 degrees
- moved D17 26.0 mm to (55.2, -6.35), turned to 270 degrees
- moved D69 25.2 mm to (292.7, 1.91), turned to 270 degrees
- moved D65 23.9 mm to (273.7, 1.91), turned to 270 degrees
- moved D73 23.7 mm to (310.5, 3.17), turned to 270 degrees
- moved D14 23.6 mm to (42.5, -5.08), turned to 270 degrees
- moved D18 23.0 mm to (58.4, -5.08), turned to 270 degrees
- moved D1 22.9 mm to (-6.35, -7.62), turned to 270 degrees
- moved D9 22.3 mm to (24.8, -6.35), turned to 270 degrees
- moved D61 22.0 mm to (254.0, 1.91), turned to 270 degrees
- moved D68 21.7 mm to (289.6, 0.64), turned to 270 degrees
- moved D21 21.0 mm to (74.3, -6.99), turned to 270 degrees
- moved D15 20.9 mm to (45.7, -3.81), turned to 270 degrees
- moved D64 20.4 mm to (270.5, 0.64), turned to 270 degrees
- moved D19 20.3 mm to (61.6, -3.81), turned to 270 degrees
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